File: Board/CH1.sch (EAGLE design)
At the start: 33 parts, among them IC3 MCP2300X/SO, IC6 74LS595D, Q1 3.6864MHz, U1 328P

Commit message: Changes to board, checked autorouter, via and trace size. ToDo: Check silk.
Parts:
- added CR1: BZT52C5V1-7-F, trigger_pcb_library:BZT52C5V1-7-F
- added CR2: BAV16W-7-F, trigger_pcb_library:BAV16W-7-F
- added SV1: (no value), con-amp-mt:L02P
Connections:
- net GND: now also CR1.21, CR2.21, LCD1.VSS, LCD2.VSS, SV1-1.S
- net VCC: now also CR1.12, CR2.12, SV1-2.S
Other:
- moved on the sheet: A3, A4, A5, C1, C2, C3, C4, C7, C8, C9, CONTRAST1, CONTRAST2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
